File: ES_SoSe_25_Schaltplan/ES_SoSe_25_Schaltplan.kicad_sch (KiCad schematic)
At the start: 22 parts

Commit message: edited scematic
Parts:
- added R9: 10kR, symbol Device:R
- added SW1: ~, symbol Switch:SW_SPST
- renumbered SW1 to SW2, SW2 to SW3, SW3 to SW4, SW4 to SW5
Connections:
- net GND: now also U3.4 (GND), U4.4 (GND), U5.4 (GND), SW1.2 (B); no longer U3.3 (GND), U4.3 (GND), U5.3 (GND)
- net VCC: now also U3.3 (Vcc), U4.3 (Vcc), U5.3 (Vcc), R9.1; no longer U3.4 (Vcc), U4.4 (Vcc), U5.4 (Vcc)
- net at A4.RST1 (RESET): now also R9.2, SW1.1 (A)
Changed lines of the file:
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@@
 	)
 	(junction
+		(at 105.41 35.56)
+		(diameter 0)
+		(color 0 0 0 0)
+	)
+	(junction
 		(at 81.28 114.3)
 		(diameter 0)
@@
 	)
 	(junction
+		(at 105.41 96.52)
+		(diameter 0)
+		(color 0 0 0 0)
+	)
+	(junction
 		(at 228.6 71.12)
 		(diameter 0)
@@
 	)
 	(junction
+		(at 91.44 114.3)
+		(diameter 0)
+		(color 0 0 0 0)
+	)
+	(junction
 		(at 172.72 99.06)
 		(diameter 0)
@@
 	(wire
 		(pts
-			(xy 111.76 43.18) (xy 111.76 49.53)
+			(xy 101.6 30.48) (xy 101.6 44.45)
 		)
 		(stroke
@@
 	(wire
 		(pts
+			(xy 105.41 95.25) (xy 105.41 96.52)
+		)
+		(stroke
+			(width 0)
+			(type default)
+		)
+	)
+	(wire
+		(pts
 			(xy 81.28 114.3) (xy 71.12 114.3)
 		)
@@
 	(wire
 		(pts
+			(xy 105.41 114.3) (xy 91.44 114.3)
+		)
+		(stroke
+			(width 0)
+			(type default)
+		)
+	)
+	(wire
+		(pts
 			(xy 167.64 118.11) (xy 167.64 137.16)
 		)
@@
 	(wire
 		(pts
-			(xy 170.18 129.54) (xy 170.18 137.16)
+			(xy 105.41 96.52) (xy 121.92 96.52)
 		)
 		(stroke
@@
 	(wire
 		(pts
-			(xy 96.52 71.12) (xy 121.92 71.12)
+			(xy 170.18 129.54) (xy 170.18 137.16)
 		)
 		(stroke
@@
 	(wire
 		(pts
-			(xy 167.64 118.11) (xy 184.15 118.11)
+			(xy 96.52 71.12) (xy 121.92 71.12)
 		)
 		(stroke
@@
 	(wire
 		(pts
-			(xy 172.72 68.58) (xy 181.61 68.58)
+			(xy 167.64 118.11) (xy 184.15 118.11)
 		)
 		(stroke
@@
 	(wire
 		(pts
-			(xy 60.96 96.52) (xy 60.96 102.87)
+			(xy 172.72 68.58) (xy 181.61 68.58)
 		)
 		(stroke
@@
 	(wire
 		(pts
-			(xy 71.12 78.74) (xy 71.12 88.9)
+			(xy 60.96 96.52) (xy 60.96 102.87)
 		)
 		(stroke
@@
 	(wire
 		(pts
-			(xy 111.76 43.18) (xy 101.6 43.18)
+			(xy 71.12 78.74) (xy 71.12 88.9)
 		)
 		(stroke
@@
 	(wire
 		(pts
+			(xy 105.41 87.63) (xy 105.41 35.56)
+		)
+		(stroke
+			(width 0)
+			(type default)
+		)
+	)
+	(wire
+		(pts
 			(xy 181.61 68.58) (xy 181.61 38.1)
 		)
@@
 	(wire
 		(pts
+			(xy 105.41 110.49) (xy 105.41 114.3)
+		)
+		(stroke
+			(width 0)
+			(type default)
+		)
+	)
+	(wire
+		(pts
 			(xy 41.91 88.9) (xy 41.91 92.71)
 		)
@@
 	(wire
 		(pts
-			(xy 101.6 43.18) (xy 101.6 30.48)
+			(xy 19.05 63.5) (xy 19.05 78.74)
 		)
 		(stroke
@@
 	(wire
 		(pts
-			(xy 19.05 63.5) (xy 19.05 78.74)
+			(xy 118.11 123.19) (xy 223.52 123.19)
 		)
 		(stroke
@@
 	(wire
 		(pts
-			(xy 118.11 123.19) (xy 223.52 123.19)
+			(xy 26.67 92.71) (xy 34.29 92.71)
 		)
 		(stroke
@@
 	(wire
 		(pts
-			(xy 26.67 92.71) (xy 34.29 92.71)
+			(xy 105.41 96.52) (xy 105.41 100.33)
 		)
 		(stroke
@@
 		(dnp no)
 		(fields_autoplaced yes)
-		(property "Reference" "SW4"
+		(property "Reference" "SW5"
 			(at 44.45 83.1849 90)
 			(effects
@@
 			(project "ES_SoSe_25_Schaltplan"
 				(path "/232146ae-6a38-4d21-b056-d9d96ad8f36d"
-					(reference "SW4")
+					(reference "SW5")
 					(unit 1)
 				)
@@
 	(symbol
 		(lib_id "Switch:SW_SPST")
-		(at 19.05 83.82 270)
+		(at 105.41 105.41 270)
 		(unit 1)
 		(exclude_from_sim no)
@@
 		(fields_autoplaced yes)
 		(property "Reference" "SW1"
+			(at 107.95 104.7749 90)
+			(effects
+				(font
+					(size 1.27 1.27)
+				)
+				(justify left)
+			)
+		)
+		(property "Value" "~"
+			(at 107.95 106.68 90)
+			(effects
+				(font
+					(size 1.27 1.27)
+				)
+				(justify left)
+			)
+		)
+		(property "Footprint" ""
+			(at 105.41 105.41 0)
+			(effects
+				(font
+					(size 1.27 1.27)
+				)
+				(hide yes)
+			)
+		)
+		(property "Datasheet" "~"
+			(at 105.41 105.41 0)
+			(effects
+				(font
+					(size 1.27 1.27)
+				)
+				(hide yes)
+			)
+		)
+		(property "Description" "Single Pole Single Throw (SPST) switch"
+			(at 105.41 105.41 0)
+			(effects
+				(font
+					(size 1.27 1.27)
+				)
+				(hide yes)
+			)
+		)
+		(pin "2"
+		)
+		(pin "1"
+		)
+		(instances
+			(project "ES_SoSe_25_Schaltplan"
+				(path "/232146ae-6a38-4d21-b056-d9d96ad8f36d"
+					(reference "SW1")
+					(unit 1)
+				)
+			)
+		)
+	)
+	(symbol
+		(lib_id "Switch:SW_SPST")
+		(at 19.05 83.82 270)
+		(unit 1)
+		(exclude_from_sim no)
+		(in_bom yes)
+		(on_board yes)
+		(dnp no)
+		(fields_autoplaced yes)
+		(property "Reference" "SW2"
 			(at 21.59 83.1849 90)
 			(effects
@@
 			(project ""
 				(path "/232146ae-6a38-4d21-b056-d9d96ad8f36d"
-					(reference "SW1")
+					(reference "SW2")
 					(unit 1)
 				)
@@
 	(symbol
 		(lib_id "power:GND")
-		(at 111.76 49.53 0)
+		(at 101.6 44.45 0)
 		(unit 1)
 		(exclude_from_sim no)
@@
 		(fields_autoplaced yes)
 		(property "Reference" "#PWR04"
-			(at 111.76 55.88 0)
+			(at 101.6 50.8 0)
 			(effects
 				(font
@@
 		)
 		(property "Value" "GND"
-			(at 111.76 54.61 0)
+			(at 101.6 49.53 0)
 			(effects
 				(font
@@
 		)
 		(property "Footprint" ""
-			(at 111.76 49.53 0)
+			(at 101.6 44.45 0)
 			(effects
 				(font
@@
 		)
 		(property "Datasheet" ""
-			(at 111.76 49.53 0)
+			(at 101.6 44.45 0)
 			(effects
 				(font
@@
 		)
 		(property "Description" "Power symbol creates a global label with name \"GND\" , ground"
-			(at 111.76 49.53 0)
+			(at 101.6 44.45 0)
 			(effects
 				(font
@@
 	)
 	(symbol
+		(lib_id "Device:R")
+		(at 105.41 91.44 0)
+		(unit 1)
+		(exclude_from_sim no)
+		(in_bom yes)
+		(on_board yes)
+		(dnp no)
+		(fields_autoplaced yes)
+		(property "Reference" "R9"
+			(at 107.95 90.1699 0)
+			(effects
+				(font
+					(size 1.27 1.27)
+				)
+				(justify left)
+			)
+		)
+		(property "Value" "10kR"
+			(at 107.95 92.7099 0)
+			(effects
+				(font
+					(size 1.27 1.27)
+				)
+				(justify left)
+			)
+		)
+		(property "Footprint" ""
+			(at 103.632 91.44 90)
+			(effects
+				(font
+					(size 1.27 1.27)
+				)
+				(hide yes)
+			)
+		)
+		(property "Datasheet" "~"
+			(at 105.41 91.44 0)
+			(effects
+				(font
+					(size 1.27 1.27)
+				)
+				(hide yes)
+			)
+		)
+		(property "Description" "Resistor"
+			(at 105.41 91.44 0)
+			(effects
+				(font
+					(size 1.27 1.27)
+				)
+				(hide yes)
+			)
+		)
+		(pin "1"
+		)
+		(pin "2"
+		)
+		(instances
+			(project "ES_SoSe_25_Schaltplan"
+				(path "/232146ae-6a38-4d21-b056-d9d96ad8f36d"
+					(reference "R9")
+					(unit 1)
+				)
+			)
+		)
+	)
+	(symbol
 		(lib_id "power:VCC")
 		(at 236.22 121.92 0)
@@
 		(dnp no)
 		(fields_autoplaced yes)
-		(property "Reference" "SW3"
+		(property "Reference" "SW4"
 			(at 36.83 83.1849 90)
 			(effects
@@
 			(project "ES_SoSe_25_Schaltplan"
 				(path "/232146ae-6a38-4d21-b056-d9d96ad8f36d"
-					(reference "SW3")
+					(reference "SW4")
 					(unit 1)
 				)
@@
 	)
 	(symbol
-		(lib_name "SSD1806_1")
 		(lib_id "es_custom_symbols:SSD1806")
 		(at 99.06 24.13 0)
@@
 	)
 	(symbol
-		(lib_name "SSD1806_1")
+		(lib_name "SSD1806_2")
 		(lib_id "es_custom_symbols:SSD1806")
 		(at 231.14 44.45 0)
@@
 		(dnp no)
 		(fields_autoplaced yes)
-		(property "Reference" "SW2"
+		(property "Reference" "SW3"
 			(at 29.21 83.1849 90)
 			(effects
@@
 			(project "ES_SoSe_25_Schaltplan"
 				(path "/232146ae-6a38-4d21-b056-d9d96ad8f36d"
-					(reference "SW2")
+					(reference "SW3")
 					(unit 1)
 				)
