File: ES_SoSe_25_Schaltplan/ES_SoSe_25_Schaltplan.kicad_sch (KiCad schematic)
At the start: 24 parts

Commit message: updated scematic
Other:
- note added: "ABS"
- note added: "Airbag"
- note added: "Blinker links"
- note added: "Blinker rechts"
- note added: "Display links"
- note added: "Display mitte"
- note added: "Display rechts"
- note added: "Fernlicht"
- note added: "RESETf"
- note added: "Scheinwerfer"
- note added: "Tempomat Set"
- note added: "Tempomat an/aus"
- note added: "Tempomat on"
- note added: "links"
- note added: "rechts"
- moved on the sheet: R4, R5, R6, R7, R8, R9
